File: justadongle/justadongle.kicad_pcb (KiCad board)
At the start: 2 copper layers, 76 x 100.5 mm, 29 parts, among them U1 SL2.1A_C6798314, U2 FSUSB42MUX, U3 LMV7219M5X/NOPB, U4 HC-USB3.0-C26, Y1 12Mhz

Commit message: redesigned the whole thingy cause of the messed up c port and additional capacitors and diodes
Parts:
- removed C8, C9: 10uf, easyeda2kicad:C0805
- removed D2, D3, D4, D5: NSR0320MW2T1G, Footprints:SOD-323_L1.8-W1.3-LS2.5-RD
- removed USB6: TYPE-C 16PIN 2MD(073), Footprints:USB-C-SMD_TYPE-C-6PIN-2MD-073
- added C12: 10uf, Footprints:C0805, F.Cu at (145.3, 131.5)
- added C13: 10uf, Footprints:C0805, F.Cu at (134.3, 77.7)
- added C14: 10uf, Footprints:C0805, F.Cu at (124.1, 132.8)
- added C15: 10uf, Footprints:C0805, F.Cu at (118.8, 137.4)
- added D10: NSR0320MW2T1G, Footprints:SOD-323_L1.8-W1.3-LS2.5-RD, F.Cu at (119.6, 144.9)
- added D11: NSR0320MW2T1G, Footprints:SOD-323_L1.8-W1.3-LS2.5-RD, F.Cu at (136.2, 125.6)
- added D6: NSR0320MW2T1G, Footprints:SOD-323_L1.8-W1.3-LS2.5-RD, F.Cu at (129.6, 147.1)
- added D7: NSR0320MW2T1G, Footprints:SOD-323_L1.8-W1.3-LS2.5-RD, F.Cu at (148.4, 147.7)
- added D8: NSR0320MW2T1G, Footprints:SOD-323_L1.8-W1.3-LS2.5-RD, F.Cu at (138.4, 135.4)
- added D9: NSR0320MW2T1G, Footprints:SOD-323_L1.8-W1.3-LS2.5-RD, F.Cu at (132.2, 136.0)
- added USB1: YTC-TC16S-128_C2927282, Footprints:TYPE-C-SMD_YTC-TC16S-128, F.Cu at (136.8, 152.1)
- C1, C2, C3, C4, C5, C6, C7: footprint easyeda2kicad:C0805 -> Footprints:C0805
- Y1: footprint easyeda2kicad:CRYSTAL-SMD_4P-L3.2-W2.5-BL -> Footprints:CAP-TH_BD5.0-P2.00-D0.8-FD
- moved C1 275.0 mm to (110.4, 69.6), turned to 180 degrees
- moved U2 269.6 mm to (134.2, 112.8), turned to 180 degrees
- moved C3 265.9 mm to (111.1, 112.0)
- moved C4 265.4 mm to (111.6, 133.7)
- moved USB5 264.9 mm to (105.1, 137.2)
- moved C2 263.5 mm to (111.1, 90.7)
- moved R1 262.2 mm to (152.8, 124.0)
- moved USB3 257.7 mm to (105.1, 94.1)
- moved USB2 257.2 mm to (105.0, 73.0)
- moved U3 256.8 mm to (140.8, 122.8), turned to 180 degrees
- moved U1 255.2 mm to (137.8, 89.2), turned to 180 degrees
- moved USB4 253.9 mm to (105.1, 115.2)
- moved R3 251.7 mm to (152.3, 112.9), turned to 90 degrees
- moved U4 248.6 mm to (137.4, 66.4)
- moved D1 248.5 mm to (134.3, 72.6)
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Routing:
- net GND: track 385.4 -> 6.39 mm, vias 4 -> 0
- net Powah: track 244.9 -> 184.0 mm, vias 4 -> 0
- net DP1: track 82.1 -> 32.0 mm
- net DM2: track 76.0 -> 34.5 mm
- net DM1: track 75.4 -> 34.4 mm
- net DP2: track 69.1 -> 36.5 mm
- net Net-(U2-HSD1+): track 90.7 -> 58.9 mm, vias 0 -> 2
- net Net-(U2-HSD1-): track 88.4 -> 57.0 mm, vias 0 -> 2
- net DP: track 45.0 -> 18.8 mm, vias 2 -> 0
- net DM : track 44.2 -> 18.8 mm, vias 2 -> 0
- net Net-(D11-A): track 0.00 -> 24.9 mm
- net Net-(D10-A): track 0.00 -> 20.5 mm
- net Net-(D5-A): track 20.0 -> 0.00 mm
- net DP3: track 66.7 -> 51.1 mm
- net DM3: track 62.3 -> 47.0 mm
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Other:
- board size 76 x 100.5 mm -> 74.2 x 92.9 mm
